File: Hardware Engineering/Digital Technology Exercise/Exercise 5/Question 1/Arduino/Arduino.brd (EAGLE design)
At the start: 100 x 80 mm, 72 parts, among them IC1 MC33269ST-5.0T3, IC2 MC33269D-5.0, IC3 ATMEGA2560-16AU, IC4 ATMEGA8U2-MU, IC5 LM358D, IC6 LP2985-33DBVR, Q1 16MHz, Q2 16MHz, T2 FDN340P, X1 DC21MMX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

Commit message: update
Parts:
- moved ADCH 156.6 mm to (82.5, 2.54)
- moved JP4 148.8 mm to (96.5, 7.62)
- moved ON 143.7 mm to (76.2, 36.8), turned to 90 degrees
- moved XIOL 143.2 mm to (95.2, 19.1), turned to 90 degrees
- moved JP3 142.1 mm to (94.0, 7.62)
- moved U$2 124.7 mm to (70.8, 38.2)
- moved JP2 124.5 mm to (96.5, 50.8)
- moved COMMUNICATION 123.4 mm to (77.5, 50.8), turned to 180 degrees
- moved RESET-EN 122.2 mm to (27.9, 15.2)
- moved C15 122.1 mm to (40.0, 17.8), turned to 270 degrees
- moved U$5 120.8 mm to (50.8, 28.3)
- moved C14 120.6 mm to (40.0, 11.4), turned to 90 degrees
- moved XIOH 119.5 mm to (95.2, 39.4), turned to 90 degrees
- moved JP1 117.1 mm to (94.0, 50.8)
- moved R1 115.0 mm to (40.0, 14.6), turned to 90 degrees
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Routing:
- net +5V: track 0.00 -> 292.7 mm, vias 0 -> 24
- net RESET: track 0.00 -> 164.2 mm, vias 0 -> 6
- net PB3: track 0.00 -> 115.5 mm, vias 0 -> 3
- net GND: track 0.00 -> 105.0 mm, vias 0 -> 47
- net PB2: track 0.00 -> 104.6 mm, vias 0 -> 3
- net PB1: track 0.00 -> 91.3 mm, vias 0 -> 3
- net ADC13: track 0.00 -> 75.2 mm, vias 0 -> 1
- net ADC14: track 0.00 -> 72.8 mm, vias 0 -> 1
- net N$3: track 0.00 -> 72.7 mm, vias 0 -> 4
- net ADC11: track 0.00 -> 71.4 mm, vias 0 -> 1
- net ADC12: track 0.00 -> 71.3 mm, vias 0 -> 1
- net ADC15: track 0.00 -> 70.6 mm, vias 0 -> 1
- net SCL: track 0.00 -> 68.5 mm, vias 0 -> 2
- net PB0: track 0.00 -> 66.4 mm, vias 0 -> 2
- net ADC10: track 0.00 -> 64.9 mm, vias 0 -> 1
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- added copper zone on layer 1, net +5V
- added copper zone on layer 16, net +5V
- added copper zone on layer 1, net GND
- added copper zone on layer 16, net GND
Other:
- board size 100 x 80 mm -> 101.6 x 53.3 mm
- board text added: "0"
- board text added: "1"
- board text added: "10"
- board text added: "11"
- board text added: "12"
- board text added: "13"
- board text added: "14"
- board text added: "15"
- board text added: "16"
- board text added: "17"
- board text added: "18"
- board text added: "19"
- board text added: "2"
- board text added: "20"
- board text added: "21"
- board text added: "22"
- board text added: "24"
- board text added: "26"
- board text added: "28"
- board text added: "3"
- board text added: "30"
- board text added: "31"
- board text added: "32"
- board text added: "33"
- board text added: "34"
- board text added: "35"
- board text added: "36"
- board text added: "37"
- board text added: "38"
- board text added: "39"
- board text added: "3V3"
- board text added: "4"
- board text added: "40"
- board text added: "41"
- board text added: "42"
- board text added: "43"
- board text added: "44"
- board text added: "45"
- board text added: "46"
- board text added: "47"
- board text added: "48"
- board text added: "49"
- board text added: "5"
- board text added: "50"
- board text added: "51"
- board text added: "52"
- board text added: "53"
- board text added: "5V"
- board text added: "6"
- board text added: "7"
- board text added: "8"
- board text added: "9"
- board text added: "ANALOG IN"
- board text added: "AREF"
- board text added: "Arduino"
- board text added: "DIGITAL"
- board text added: "GND"
- board text added: "ITALY"
- board text added: "L"
- board text added: "MADE IN"
- board text added: "MEGA 2560"
- board text added: "MEGAXL"
- board text added: "PC1"
- board text added: "PC2"
- board text added: "PWM"
- board text added: "RESET"
- board text added: "RX"
- board text added: "RX1"
- board text added: "RX2"
- board text added: "RX3"
- board text added: "SCL"
- board text added: "SDA"
- board text added: "TM"
- board text added: "TX"
- board text added: "TX1"
- board text added: "TX2"
- board text added: "TX3"
- board text added: "VIN"
- board text added: "designed by"
- board text added: "tinker it"
- board text added: "www.arduino.cc"
