File: Hardware Engineering/Lab Project/Parking Lot System Main Board/Parking Lot System Main Board.sch (EAGLE design)
At the start: 15 parts, among them IC1 NE555

Commit message: update
Parts:
- removed U$1: CYPHER2022, CYPHER:CYPHER2022
- added CYPHER: CYPHER2022, CYPHER:CYPHER2022
Connections:
- net CLK: now also CYPHER.CLK; no longer U$1.CLK
- net GND: now also CYPHER.GND; no longer U$1.GND
- net N$1: now also CYPHER.CAR_ENTER; no longer U$1.CAR_ENTER
- net N$10: now also CYPHER.INDICATOR_GREEN; no longer U$1.INDICATOR_GREEN
- net N$12: now also CYPHER.INDICATOR_CLOSE; no longer U$1.INDICATOR_CLOSE
- net N$13: now also CYPHER.DIGIT_00; no longer U$1.DIGIT_00
- net N$14: now also CYPHER.DIGIT_01; no longer U$1.DIGIT_01
- net N$15: now also CYPHER.DIGIT_02; no longer U$1.DIGIT_02
- net N$16: now also CYPHER.DIGIT_03; no longer U$1.DIGIT_03
- net N$17: now also CYPHER.DIGIT_04; no longer U$1.DIGIT_04
- net N$18: now also CYPHER.DIGIT_05; no longer U$1.DIGIT_05
- net N$19: now also CYPHER.DIGIT_06; no longer U$1.DIGIT_06
- net N$2: now also CYPHER.RESET; no longer U$1.RESET
- net N$20: now also CYPHER.DIGIT_10; no longer U$1.DIGIT_10
- net N$21: now also CYPHER.DIGIT_11; no longer U$1.DIGIT_11
- net N$22: now also CYPHER.DIGIT_12; no longer U$1.DIGIT_12
- net N$23: now also CYPHER.DIGIT_13; no longer U$1.DIGIT_13
- net N$24: now also CYPHER.DIGIT_14; no longer U$1.DIGIT_14
- net N$25: now also CYPHER.DIGIT_15; no longer U$1.DIGIT_15
- net N$26: now also CYPHER.DIGIT_26; no longer U$1.DIGIT_26
- net N$27: now also CYPHER.DIGIT_16; no longer U$1.DIGIT_16
- net N$28: now also CYPHER.DIGIT_20; no longer U$1.DIGIT_20
- net N$29: now also CYPHER.DIGIT_21; no longer U$1.DIGIT_21
- net N$30: now also CYPHER.DIGIT_22; no longer U$1.DIGIT_22
- net N$31: now also CYPHER.DIGIT_23; no longer U$1.DIGIT_23
- net N$32: now also CYPHER.DIGIT_24; no longer U$1.DIGIT_24
- net N$33: now also CYPHER.DIGIT_25; no longer U$1.DIGIT_25
- net N$5: now also CYPHER.CAR_LEAVE; no longer U$1.CAR_LEAVE
- net N$6: now also CYPHER.READY; no longer U$1.READY
- net N$8: now also CYPHER.GATE_OPEN; no longer U$1.GATE_OPEN
- net N$9: now also CYPHER.GATE_CLOSE; no longer U$1.GATE_CLOSE
- net VIN: now also CYPHER.VIN; no longer U$1.VIN
Other:
- moved on the sheet: C1, C2, C3, D1, D2, DIGIT1-1, DIGIT1-2, DIGIT1-3, DIGIT1-4, DIGIT1-5, DIGIT1-6, DIGIT1-7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
